File: HX-1/power_clock_io.kicad_sch (KiCad schematic)
At the start: 27 parts, among them Y1 16MHz

Commit message: change schematic file name and doc, script references
Parts:
- removed C1, C10, C11, C12, C13, C17, C2, C3, C4, C5, C6, C7, C8, C9: 100nF, Capacitor_SMD:C_0402_1005Metric, symbol Device:C
- removed C14: 10uF, Capacitor_SMD:C_0603_1608Metric, symbol Device:C
- removed C15: 1uF, Capacitor_SMD:C_0603_1608Metric, symbol Device:C
- removed C16, C19: 1uF, Capacitor_SMD:C_0402_1005Metric, symbol Device:C
- removed C18: 10nF, Capacitor_SMD:C_0603_1608Metric, symbol Device:C
- removed C22, C23: 10pF, Capacitor_SMD:C_0603_1608Metric, symbol Device:C
- removed FB1: 100R, Resistor_SMD:R_0805_2012Metric, symbol Device:FerriteBead
- removed H1, H2, H3, H4: MountingHole_Pad, MountingHole:MountingHole_3.2mm_M3_Pad, symbol Mechanical:MountingHole_Pad
- removed Y1: 16MHz, Crystal:Crystal_SMD_3225-4Pin_3.2x2.5mm, symbol Device:Crystal_GND24
Other:
- note removed: "(Load_C (9pF) - Stray_C (~4pF) ) * 2 = 10 pF"
- note removed: "Bulk Decoupling"
- note removed: "For VDDUSB filtering"
- note removed: "HSE Clock"
- note removed: "MCU Analog Filtering"
- note removed: "MCU VDD Filtering"
- note removed: "Mounting Holes"
- note removed: "one C for each VDD/VBAT"
- note removed: "page 162. VDDA and VREF chosen to be connected externally."
