File: HX-1/communication_power.kicad_sch (KiCad schematic)
At the start: 31 parts, among them J1 USB_C_Receptacle_USB2.0_16P, J2 Conn_01x02_Socket, U2 USBLC6-2SC6, U3 XC6206P332MR-G, U4 LSM6DS3

Commit message: add assembly files, fix reference designators
Parts:
- BZ1: LCSC C781883 -> (none); LCSC PN (none) -> C781883
- D3, D7: LCSC C2286 -> (none); LCSC PN (none) -> C2286
- J2: LCSC PN (none) -> C131337
- U4: LCSC C126672 -> (none); LCSC PN (none) -> C95230
- renumbered D5 to D4, D4 to D5

Commit message: change LSM6DS to version compat with jlcpcb economic pcba
Parts:
- U4: value LSM6DS3 -> LSM6DSRTR; LCSC PN C95230 -> C784817
Changed lines of the file:
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@@
 			)
 		)
-		(property "Value" "LSM6DS3"
+		(property "Value" "LSM6DSRTR"
 			(at 112.268 119.634 0)
 			(effects
@@
 			)
 		)
-		(property "LCSC PN" "C95230"
+		(property "LCSC PN" "C784817"
 			(at 111.76 115.57 0)
 			(effects
